Commit message: fix some bug

File: urdfs/d1_description/xacro/robot.xacro (robot description, xacro)
@@ -3,47 +3,47 @@
     xmlns:xacro="http://www.ros.org/wiki/xacro">
     <xacro:arg name="hw_env" default="none" />
-    <xacro:include filename="$(find d1_description)/xacro/ros2control.xacro"/>
+    <xacro:include filename="$(find d1_description)/xacro/ros2control.xacro" />
     <xacro:ros2control hw_env="$(arg hw_env)" />
-    <xacro:include filename="$(find d1h_description)/xacro/materials.xacro"/>
-    <xacro:include filename="$(find d1h_description)/xacro/single_robot.xacro"/>
+    <xacro:include filename="$(find d1h_description)/xacro/materials.xacro" />
+    <xacro:include filename="$(find d1h_description)/xacro/single_robot.xacro" />
     <link name="base_link">
         <visual>
-            <origin rpy="0 0 0" xyz="0 0 0"/>
+            <origin rpy="0 0 0" xyz="0 0 0" />
             <geometry>
-                <box size="0.001 0.001 0.001"/>
+                <box size="0.001 0.001 0.001" />
             </geometry>
         </visual>
         <inertial>
-            <mass value="0.001"/>
-            <origin rpy="0 0 0" xyz="0 0 0"/>
-            <inertia ixx="0.0001" ixy="0" ixz="0" iyy="0.0001" iyz="0" izz="0.0001"/>
+            <mass value="0.001" />
+            <origin rpy="0 0 0" xyz="0 0 0" />
+            <inertia ixx="0.0001" ixy="0" ixz="0" iyy="0.0001" iyz="0" izz="0.0001" />
         </inertial>
     </link>
     <link name="imu_link">
         <inertial>
-            <mass value="0.001"/>
-            <origin rpy="0 0 0" xyz="0 0 0"/>
-            <inertia ixx="0.0001" ixy="0" ixz="0" iyy="0.0001" iyz="0" izz="0.0001"/>
+            <mass value="0.001" />
+            <origin rpy="0 0 0" xyz="0 0 0" />
+            <inertia ixx="0.0001" ixy="0" ixz="0" iyy="0.0001" iyz="0" izz="0.0001" />
         </inertial>
         <visual>
-            <origin rpy="0 0 0" xyz="0 0 0"/>
+            <origin rpy="0 0 0" xyz="0 0 0" />
             <geometry>
-                <box size="0.001 0.001 0.001"/>
+                <box size="0.001 0.001 0.001" />
             </geometry>
-            <material name="red"/>
+            <material name="red" />
         </visual>
         <collision>
-            <origin rpy="0 0 0" xyz="0 0 0"/>
+            <origin rpy="0 0 0" xyz="0 0 0" />
             <geometry>
-                <box size=".001 .001 .001"/>
+                <box size=".001 .001 .001" />
             </geometry>
         </collision>
     </link>
     <joint name="imu_joint" type="fixed">
-        <parent link="base_link"/>
-        <child link="imu_link"/>
-        <origin rpy="0 0 0" xyz="0 0 0"/>
+        <parent link="base_link" />
+        <child link="imu_link" />
+        <origin rpy="0 0 0" xyz="0 0 0" />
     </joint>
-    <xacro:single_robot name="F" x_offset="0.1875"/>
-    <xacro:single_robot name="R" x_offset="-0.1875"/>
+    <xacro:single_robot name="F" x_offset="0.1875" />
+    <xacro:single_robot name="R" x_offset="-0.1875" />
 </robot>
